Commit message: fixed hardware interace but bot is spinning wrong

File: src/robot/urdf/control/ros2_control.xacro (robot description, xacro)
@@ -1,40 +1,19 @@
 <?xml version="1.0"?>
 <robot xmlns:xacro="http://www.ros.org/wiki/xacro">
-<!-- <ros2_control name="RealRobot" type="system">
-    <hardware>
-        <plugin>diffdrive_arduino/DiffDriveArduino</plugin>
-        <param name="left_wheel_name">left_wheel_joint</param>
-        <param name="right_wheel_name">right_wheel_joint</param>
-        <param name="loop_rate">30</param>
-        <param name="device">/dev/ttyACM0</param>
-        <param name="baud_rate">57600</param>
-        <param name="timeout">1000</param>
-        <param name="enc_counts_per_rev">3436</param>
-    </hardware>
-    <joint name="left_wheel_joint">
-        <command_interface name="velocity">
-            <param name="min">-10</param>
-            <param name="max">10</param>
-        </command_interface>
-        <state_interface name="velocity"/>
-        <state_interface name="position"/>
-    </joint>
-    <joint name="right_wheel_joint">
-        <command_interface name="velocity">
-            <param name="min">-10</param>
-            <param name="max">10</param>
-        </command_interface>
-        <state_interface name="velocity"/>
-        <state_interface name="position"/>
-    </joint>
-</ros2_control> -->
-    <ros2_control name="GazeboSystem" type="system">
+    <ros2_control name="RealRobot" type="system">
         <hardware>
-            <plugin>gazebo_ros2_control/GazeboSystem</plugin>
+            <plugin>diffdrive_arduino/DiffDriveArduino</plugin>
+            <param name="left_wheel_name">left_wheel_joint</param>
+            <param name="right_wheel_name">right_wheel_joint</param>
+            <param name="loop_rate">30</param>
+            <param name="device">/dev/ttyACM0</param>
+            <param name="baud_rate">57600</param>
+            <param name="timeout">1000</param>
+            <param name="enc_counts_per_rev">560</param>
         </hardware>
         <joint name="left_wheel_joint">
             <command_interface name="velocity">
-                <param name="min">-100</param>
-                <param name="max">100</param>
+                <param name="min">-10</param>
+                <param name="max">10</param>
             </command_interface>
             <state_interface name="velocity"/>
@@ -43,6 +22,6 @@
         <joint name="right_wheel_joint">
             <command_interface name="velocity">
-                <param name="min">-100</param>
-                <param name="max">100</param>
+                <param name="min">-10</param>
+                <param name="max">10</param>
             </command_interface>
             <state_interface name="velocity"/>

File: src/robot/urdf/robot.urdf.xacro (robot description, xacro)
@@ -5,7 +5,7 @@
 <link name="base_link">
   <inertial>
-    <origin xyz="-0.07617652640143699 0.0009658129509204017 0.0007548948976041592" rpy="0 0 0"/>
+    <origin xyz="-0.0004442275486858486 -0.027763800307559608 0.04075489489760404" rpy="0 0 0"/>
     <mass value="1.449043338359083"/>
-    <inertia ixx="0.013382" iyy="0.012" izz="0.01271" ixy="-0.0" iyz="-0.0" ixz="-0.000167"/>
+    <inertia ixx="0.012" iyy="0.013382" izz="0.01271" ixy="0.0" iyz="-0.000167" ixz="0.0"/>
   </inertial>
   <visual>
@@ -23,55 +23,55 @@
   </collision>
 </link>
-<link name="right_wheel">
+<link name="right_wheel_1">
   <inertial>
-    <origin xyz="-1.7552218505301198e-06 0.027427365846597315 1.782423703911018e-07" rpy="0 0 0"/>
+    <origin xyz="-0.027427780444362282 -2.029127972526094e-06 1.7824236945435112e-07" rpy="0 0 0"/>
     <mass value="0.05590599422944014"/>
-    <inertia ixx="3.2e-05" iyy="5e-05" izz="3.2e-05" ixy="-0.0" iyz="0.0" ixz="-0.0"/>
+    <inertia ixx="5e-05" iyy="3.2e-05" izz="3.2e-05" ixy="0.0" iyz="-0.0" ixz="-0.0"/>
   </inertial>
   <visual>
-    <origin xyz="0.047514 -0.124767 0.077546" rpy="0 0 0"/>
+    <origin xyz="0.124245 -0.000899 0.037546" rpy="0 0 0"/>
     <geometry>
-      <mesh filename="file://$(find robot)/meshes/Wheel_1_1.stl" scale="0.001 0.001 0.001"/>
+      <mesh filename="file://$(find robot)/meshes/right_wheel_1.stl" scale="0.001 0.001 0.001"/>
     </geometry>
     <material name="silver"/>
   </visual>
   <collision>
-    <origin xyz="0.047514 -0.124767 0.077546" rpy="0 0 0"/>
+    <origin xyz="0.124245 -0.000899 0.037546" rpy="0 0 0"/>
     <geometry>
-      <mesh filename="file://$(find robot)/meshes/Wheel_1_1.stl" scale="0.001 0.001 0.001"/>
+      <mesh filename="file://$(find robot)/meshes/right_wheel_1.stl" scale="0.001 0.001 0.001"/>
     </geometry>
   </collision>
 </link>
-<link name="left_wheel">
+<link name="left_wheel_1">
   <inertial>
-    <origin xyz="-1.7552218502803196e-06 -0.02742790766788944 1.5656025187382738e-07" rpy="0 0 0"/>
+    <origin xyz="0.027427493070124417 -2.0291279724919415e-06 1.5656025283833364e-07" rpy="0 0 0"/>
     <mass value="0.05590599422944014"/>
-    <inertia ixx="3.2e-05" iyy="5e-05" izz="3.2e-05" ixy="0.0" iyz="0.0" ixz="0.0"/>
+    <inertia ixx="5e-05" iyy="3.2e-05" izz="3.2e-05" ixy="-0.0" iyz="0.0" ixz="-0.0"/>
   </inertial>
   <visual>
-    <origin xyz="0.047514 0.122833 0.077546" rpy="0 0 0"/>
+    <origin xyz="-0.123355 -0.000899 0.037546" rpy="0 0 0"/>
     <geometry>
-      <mesh filename="file://$(find robot)/meshes/Wheel_2_1.stl" scale="0.001 0.001 0.001"/>
+      <mesh filename="file://$(find robot)/meshes/left_wheel_1.stl" scale="0.001 0.001 0.001"/>
     </geometry>
     <material name="silver"/>
   </visual>
   <collision>
-    <origin xyz="0.047514 0.122833 0.077546" rpy="0 0 0"/>
+    <origin xyz="-0.123355 -0.000899 0.037546" rpy="0 0 0"/>
     <geometry>
-      <mesh filename="file://$(find robot)/meshes/Wheel_2_1.stl" scale="0.001 0.001 0.001"/>
+      <mesh filename="file://$(find robot)/meshes/left_wheel_1.stl" scale="0.001 0.001 0.001"/>
     </geometry>
   </collision>
 </link>
 <joint name="right_wheel_joint" type="continuous">
-  <origin xyz="-0.047514 0.124767 -0.077546" rpy="0 0 0"/>
+  <origin xyz="-0.124245 0.000899 -0.037546" rpy="0 0 0"/>
   <parent link="base_link"/>
-  <child link="right_wheel"/>
-  <axis xyz="-0.0 1.0 0.0"/>
+  <child link="right_wheel_1"/>
+  <axis xyz="-1.0 -0.0 -0.0"/>
 </joint>
 <joint name="left_wheel_joint" type="continuous">
-  <origin xyz="-0.047514 -0.122833 -0.077546" rpy="0 0 0"/>
+  <origin xyz="0.123355 0.000899 -0.037546" rpy="0 0 0"/>
   <parent link="base_link"/>
-  <child link="left_wheel"/>
-  <axis xyz="-0.0 -1.0 -0.0"/>
+  <child link="left_wheel_1"/>
+  <axis xyz="1.0 -0.0 -0.0"/>
 </joint>
 </robot>

File: src/robot/urdf/robot_core.urdf.xacro (robot description, xacro)
@@ -3,5 +3,12 @@
 <xacro:include filename="$(find robot)/urdf/robot.urdf.xacro" />
 <!-- <xacro:include filename="$(find robot)/urdf/sensors/lidar.xacro" /> -->
-<xacro:include filename="$(find robot)/urdf/control/gazebo_control.xacro" />
-<!-- <xacro:include filename="$(find robot)/urdf/control/ros2_control.xacro" /> -->
+<!-- <xacro:include filename="$(find robot)/urdf/control/gazebo_control.xacro" /> -->
+<xacro:include filename="$(find robot)/urdf/control/ros2_control.xacro" />
+<!--
+<xacro:if value="$(arg use_ros2_control)">
+    <xacro:include filename="$(find robot)/urdf/control/ros2_control.xacro" />
+</xacro:if>
+<xacro:unless value="$(arg use_ros2_control)">
+    <xacro:include filename="$(find robot)/urdf/control/gazebo_control.xacro" />
+</xacro:unless> -->
 </robot>
