Commit message: modified chassis mesh files and remade robot, still working on wheels and lidar origins

File: src/robot/urdf/control/gazebo_control.xacro (robot description, xacro)
@@ -6,6 +6,6 @@
             <left_joint>left_wheel_joint</left_joint>
             <right_joint>right_wheel_joint</right_joint>
-            <wheel_separation>0.297</wheel_separation>
-            <wheel_diameter>0.066</wheel_diameter>
+            <wheel_separation>0.31</wheel_separation>
+            <wheel_diameter>0.07</wheel_diameter>
             <!-- Limits -->
             <max_wheel_torque>200</max_wheel_torque>

File: src/robot/urdf/control/ros2_control.xacro (robot description, xacro)
@@ -1,5 +1,5 @@
 <?xml version="1.0"?>
 <robot xmlns:xacro="http://www.ros.org/wiki/xacro">
-<ros2_control name="RealRobot" type="system">
+<!-- <ros2_control name="RealRobot" type="system">
     <hardware>
         <plugin>diffdrive_arduino/DiffDriveArduino</plugin>
@@ -28,6 +28,6 @@
         <state_interface name="position"/>
     </joint>
-</ros2_control>
-    <!-- <ros2_control name="GazeboSystem" type="system">
+</ros2_control> -->
+    <ros2_control name="GazeboSystem" type="system">
         <hardware>
             <plugin>gazebo_ros2_control/GazeboSystem</plugin>
@@ -35,6 +35,6 @@
         <joint name="left_wheel_joint">
             <command_interface name="velocity">
-                <param name="min">-10</param>
-                <param name="max">10</param>
+                <param name="min">-100</param>
+                <param name="max">100</param>
             </command_interface>
             <state_interface name="velocity"/>
@@ -43,11 +43,11 @@
         <joint name="right_wheel_joint">
             <command_interface name="velocity">
-                <param name="min">-10</param>
-                <param name="max">10</param>
+                <param name="min">-100</param>
+                <param name="max">100</param>
             </command_interface>
             <state_interface name="velocity"/>
             <state_interface name="position"/>
         </joint>
-    </ros2_control> -->
+    </ros2_control>
     <gazebo>
         <plugin name="gazebo_ros2_control" filename="libgazebo_ros2_control.so">

File: src/robot/urdf/properties.xacro (robot description, xacro)
@@ -1,23 +1,30 @@
 <?xml version="1.0" ?>
 <robot name="ros" xmlns:xacro="http://www.ros.org/wiki/xacro" >
-<xacro:property name="body_color" value="Gazebo/Silver" />
-<gazebo reference="base_link">
+<!-- <xacro:property name="body_color" value="Gazebo/Silver" /> -->
+<gazebo reference="chassis_link">
   <material>Gazebo/Green</material>
-  <mu1>0.2</mu1>
+  <!-- <mu1>0.2</mu1>
   <mu2>0.2</mu2>
   <selfCollide>true</selfCollide>
-  <gravity>true</gravity>
+  <gravity>true</gravity> -->
 </gazebo>
-<gazebo reference="Wheel_1_1">
+<gazebo reference="right_wheel">
   <material>Gazebo/Black</material>
   <mu1>0.2</mu1>
   <mu2>0.2</mu2>
-  <selfCollide>true</selfCollide>
+  <!-- <selfCollide>true</selfCollide> -->
 </gazebo>
-<gazebo reference="Wheel_2_1">
+<gazebo reference="left_wheel">
   <material>Gazebo/Black</material>
   <mu1>0.2</mu1>
   <mu2>0.2</mu2>
-  <selfCollide>true</selfCollide>
+  <!-- <selfCollide>true</selfCollide> -->
+</gazebo>
+<gazebo reference="lidar_link">
+  <material>Gazebo/Black</material>
+  <!-- <mu1>0.2</mu1> -->
+  <!-- <mu2>0.2</mu2> -->
+  <!-- <selfCollide>true</selfCollide> -->
+  <!-- <gravity>true</gravity> -->
 </gazebo>
 </robot>

File: src/robot/urdf/robot.urdf.xacro (robot description, xacro)
@@ -4,72 +4,89 @@
 <xacro:include filename="$(find robot)/urdf/properties.xacro" />
 <link name="base_link">
+</link>
+<!-- BASE_FOOTPRINT LINK -->
+<joint name="base_footprint_joint" type="fixed">
+    <parent link="base_link"/>
+    <child link="base_footprint"/>
+    <origin xyz="0 0 0" rpy="0 0 0"/>
+</joint>
+<link name="base_footprint">
+</link>
+<link name="chassis_link">
   <inertial>
-    <origin xyz="0.0025530868570427627 0.07969811180367155 0.0007548948976046698" rpy="0 0 0"/>
-    <mass value="1.449043338359083"/>
-    <inertia ixx="0.012" iyy="0.013382" izz="0.01271" ixy="0.0" iyz="0.000167" ixz="-0.0"/>
+    <origin xyz="0.0005529614189068058 0.14968759146166039 0.0010740992367894852" rpy="0 0 0"/>
+    <mass value="1.2745335608269892"/>
+    <inertia ixx="0.008772" iyy="0.010315" izz="0.012456" ixy="0.0" iyz="-0.000402" ixz="-0.0"/>
+  </inertial>
+  <visual>
+    <origin xyz="0 0 0" rpy="0 0 -${pi/2}"/>
+    <geometry>
+      <mesh filename="file://$(find robot)/meshes/chassis/base_link.stl" scale="0.001 0.001 0.001"/>
+    </geometry>
+    <material name="silver"/>
+  </visual>
+  <collision>
+    <origin xyz="0 0 0" rpy="0 0 -${pi/2}"/>
+    <geometry>
+      <mesh filename="file://$(find robot)/meshes/chassis/base_link.stl" scale="0.001 0.001 0.001"/>
+    </geometry>
+  </collision>
+</link>
+<link name="right_wheel">
+  <inertial>
+    <origin xyz="1.0841058295907897e-08 -2.1769788347466894e-06 -0.0005723632427566792" rpy="0 0 0"/>
+    <mass value="0.05590599422944008"/>
+    <inertia ixx="3.2e-05" iyy="3.2e-05" izz="5e-05" ixy="-0.0" iyz="-0.0" ixz="0.0"/>
+  </inertial>
+  <visual>
+    <origin xyz="0 0 0" rpy="${pi/2} 0 0"/>
+    <geometry>
+      <mesh filename="file://$(find robot)/meshes/wheel/base_link.stl" scale="0.001 0.001 0.001"/>
+    </geometry>
+    <material name="silver"/>
+  </visual>
+  <collision>
+    <origin xyz="0 0 0" rpy="${pi/2} 0 0"/>
+    <geometry>
+      <mesh filename="file://$(find robot)/meshes/wheel/base_link.stl" scale="0.001 0.001 0.001"/>
+    </geometry>
+  </collision>
+</link>
+<link name="left_wheel">
+  <inertial>
+    <origin xyz="1.0841058295907897e-08 -2.1769788347466894e-06 -0.0005723632427566792" rpy="0 0 0"/>
+    <mass value="0.05590599422944008"/>
+    <inertia ixx="3.2e-05" iyy="3.2e-05" izz="5e-05" ixy="-0.0" iyz="-0.0" ixz="0.0"/>
   </inertial>
   <visual>
     <origin xyz="0 0 0" rpy="0 0 0"/>
     <geometry>
-      <mesh filename="$(find robot)/meshes/base_link.stl" scale="0.001 0.001 0.001"/>
+      <mesh filename="file://$(find robot)/meshes/wheel/base_link.stl" scale="0.001 0.001 0.001"/>
     </geometry>
-    <material name="green"/>
+    <material name="silver"/>
   </visual>
   <collision>
     <origin xyz="0 0 0" rpy="0 0 0"/>
     <geometry>
-      <mesh filename="$(find robot)/meshes/base_link.stl" scale="0.001 0.001 0.001"/>
+      <mesh filename="file://$(find robot)/meshes/wheel/base_link.stl" scale="0.001 0.001 0.001"/>
     </geometry>
   </collision>
 </link>
-<link name="Wheel_1_1">
-  <inertial>
-    <origin xyz="0.027427639752719224 2.340624085342413e-06 1.7824236978047914e-07" rpy="0 0 0"/>
-    <mass value="0.05590599422944014"/>
-    <inertia ixx="5e-05" iyy="3.2e-05" izz="3.2e-05" ixy="0.0" iyz="0.0" ixz="0.0"/>
-  </inertial>
-  <visual>
-    <origin xyz="-0.126354 -0.051035 0.077546" rpy="0 0 0"/>
-    <geometry>
-      <mesh filename="$(find robot)/meshes/Wheel_1_1.stl" scale="0.001 0.001 0.001"/>
-    </geometry>
-    <material name="black"/>
-  </visual>
-  <collision>
-    <origin xyz="-0.126354 -0.051035 0.077546" rpy="0 0 0"/>
-    <geometry>
-      <mesh filename="$(find robot)/meshes/Wheel_1_1.stl" scale="0.001 0.001 0.001"/>
-    </geometry>
-  </collision>
-</link>
-<link name="Wheel_2_1">
-  <inertial>
-    <origin xyz="-0.02742763376176742 2.34062408542568e-06 1.5656025319221722e-07" rpy="0 0 0"/>
-    <mass value="0.05590599422944014"/>
-    <inertia ixx="5e-05" iyy="3.2e-05" izz="3.2e-05" ixy="-0.0" iyz="-0.0" ixz="0.0"/>
-  </inertial>
-  <visual>
-    <origin xyz="0.121246 -0.051035 0.077546" rpy="0 0 0"/>
-    <geometry>
-      <mesh filename="$(find robot)/meshes/Wheel_2_1.stl" scale="0.001 0.001 0.001"/>
-    </geometry>
-    <material name="black"/>
-  </visual>
-  <collision>
-    <origin xyz="0.121246 -0.051035 0.077546" rpy="0 0 0"/>
-    <geometry>
-      <mesh filename="$(find robot)/meshes/Wheel_2_1.stl" scale="0.001 0.001 0.001"/>
-    </geometry>
-  </collision>
-</link>
+<joint name="chassis_joint" type="fixed">
+    <parent link="base_link"/>
+    <child link="chassis_link"/>
+    <origin xyz="-0.12 0 0.015"/>
+</joint>
 <joint name="right_wheel_joint" type="continuous">
-  <origin xyz="0.126354 0.051035 -0.077546" rpy="0 0 0"/>
-  <parent link="base_link"/>
-  <child link="Wheel_1_1"/>
+  <origin xyz="0.119 -0.1538 -0.059" rpy="0 0 0"/>
+  <parent link="chassis_link"/>
+  <child link="right_wheel"/>
+  <axis xyz="0 1 0"/>
 </joint>
 <joint name="left_wheel_joint" type="continuous">
-  <origin xyz="-0.121246 0.051035 -0.077546" rpy="0 0 0"/>
-  <parent link="base_link"/>
-  <child link="Wheel_2_1"/>
+  <origin xyz="0.119 -0.1538 0.059" rpy="0 0 0"/>
+  <parent link="chassis_link"/>
+  <child link="left_wheel"/>
+  <axis xyz="0 -1 0"/>
 </joint>
 </robot>

File: src/robot/urdf/robot_core.urdf.xacro (robot description, xacro)
@@ -1,5 +1,6 @@
 <?xml version="1.0" ?>
-<robot name="ros" xmlns:xacro="http://www.ros.org/wiki/xacro" >
+<robot name="rina" xmlns:xacro="http://www.ros.org/wiki/xacro" >
 <xacro:include filename="$(find robot)/urdf/robot.urdf.xacro" />
+<xacro:include filename="$(find robot)/urdf/sensors/lidar.xacro" />
 <!-- <xacro:include filename="$(find robot)/urdf/control/gazebo_control.xacro" /> -->
 <xacro:include filename="$(find robot)/urdf/control/ros2_control.xacro" />

Commit message: finally working however bot's forward and rotation are flipped, need to fix in fusion360

File: src/robot/urdf/control/gazebo_control.xacro (robot description, xacro)
@@ -6,5 +6,5 @@
             <left_joint>left_wheel_joint</left_joint>
             <right_joint>right_wheel_joint</right_joint>
-            <wheel_separation>0.31</wheel_separation>
+            <wheel_separation>0.3048</wheel_separation>
             <wheel_diameter>0.07</wheel_diameter>
             <!-- Limits -->

File: src/robot/urdf/properties.xacro (robot description, xacro)
@@ -1,22 +1,22 @@
 <?xml version="1.0" ?>
 <robot name="ros" xmlns:xacro="http://www.ros.org/wiki/xacro" >
-<!-- <xacro:property name="body_color" value="Gazebo/Silver" /> -->
-<gazebo reference="chassis_link">
-  <material>Gazebo/Green</material>
-  <!-- <mu1>0.2</mu1>
+<xacro:property name="body_color" value="Gazebo/Silver" />
+<gazebo reference="base_link">
+  <material>${body_color}</material>
+  <mu1>0.2</mu1>
   <mu2>0.2</mu2>
-  <selfCollide>true</selfCollide>
+  <!-- <selfCollide>true</selfCollide>
   <gravity>true</gravity> -->
 </gazebo>
 <gazebo reference="right_wheel">
   <material>Gazebo/Black</material>
-  <mu1>0.2</mu1>
-  <mu2>0.2</mu2>
+  <!-- <mu1>0.2</mu1>
+  <mu2>0.2</mu2> -->
   <!-- <selfCollide>true</selfCollide> -->
 </gazebo>
 <gazebo reference="left_wheel">
   <material>Gazebo/Black</material>
-  <mu1>0.2</mu1>
-  <mu2>0.2</mu2>
+  <!-- <mu1>0.2</mu1>
+  <mu2>0.2</mu2> -->
   <!-- <selfCollide>true</selfCollide> -->
 </gazebo>

File: src/robot/urdf/robot.urdf.xacro (robot description, xacro)
@@ -4,63 +4,13 @@
 <xacro:include filename="$(find robot)/urdf/properties.xacro" />
 <link name="base_link">
-</link>
-<!-- BASE_FOOTPRINT LINK -->
-<joint name="base_footprint_joint" type="fixed">
-    <parent link="base_link"/>
-    <child link="base_footprint"/>
-    <origin xyz="0 0 0" rpy="0 0 0"/>
-</joint>
-<link name="base_footprint">
-</link>
-<link name="chassis_link">
   <inertial>
-    <origin xyz="0.0005529614189068058 0.14968759146166039 0.0010740992367894852" rpy="0 0 0"/>
-    <mass value="1.2745335608269892"/>
-    <inertia ixx="0.008772" iyy="0.010315" izz="0.012456" ixy="0.0" iyz="-0.000402" ixz="-0.0"/>
-  </inertial>
-  <visual>
-    <origin xyz="0 0 0" rpy="0 0 -${pi/2}"/>
-    <geometry>
-      <mesh filename="file://$(find robot)/meshes/chassis/base_link.stl" scale="0.001 0.001 0.001"/>
-    </geometry>
-    <material name="silver"/>
-  </visual>
-  <collision>
-    <origin xyz="0 0 0" rpy="0 0 -${pi/2}"/>
-    <geometry>
-      <mesh filename="file://$(find robot)/meshes/chassis/base_link.stl" scale="0.001 0.001 0.001"/>
-    </geometry>
-  </collision>
-</link>
-<link name="right_wheel">
-  <inertial>
-    <origin xyz="1.0841058295907897e-08 -2.1769788347466894e-06 -0.0005723632427566792" rpy="0 0 0"/>
-    <mass value="0.05590599422944008"/>
-    <inertia ixx="3.2e-05" iyy="3.2e-05" izz="5e-05" ixy="-0.0" iyz="-0.0" ixz="0.0"/>
-  </inertial>
-  <visual>
-    <origin xyz="0 0 0" rpy="${pi/2} 0 0"/>
-    <geometry>
-      <mesh filename="file://$(find robot)/meshes/wheel/base_link.stl" scale="0.001 0.001 0.001"/>
-    </geometry>
-    <material name="silver"/>
-  </visual>
-  <collision>
-    <origin xyz="0 0 0" rpy="${pi/2} 0 0"/>
-    <geometry>
-      <mesh filename="file://$(find robot)/meshes/wheel/base_link.stl" scale="0.001 0.001 0.001"/>
-    </geometry>
-  </collision>
-</link>
-<link name="left_wheel">
-  <inertial>
-    <origin xyz="1.0841058295907897e-08 -2.1769788347466894e-06 -0.0005723632427566792" rpy="0 0 0"/>
-    <mass value="0.05590599422944008"/>
-    <inertia ixx="3.2e-05" iyy="3.2e-05" izz="5e-05" ixy="-0.0" iyz="-0.0" ixz="0.0"/>
+    <origin xyz="-0.07617652640143699 0.0009658129509204017 0.0007548948976041592" rpy="0 0 0"/>
+    <mass value="1.449043338359083"/>
+    <inertia ixx="0.013382" iyy="0.012" izz="0.01271" ixy="-0.0" iyz="-0.0" ixz="-0.000167"/>
   </inertial>
   <visual>
     <origin xyz="0 0 0" rpy="0 0 0"/>
     <geometry>
-      <mesh filename="file://$(find robot)/meshes/wheel/base_link.stl" scale="0.001 0.001 0.001"/>
+      <mesh filename="file://$(find robot)/meshes/base_link.stl" scale="0.001 0.001 0.001"/>
     </geometry>
     <material name="silver"/>
@@ -69,24 +19,59 @@
     <origin xyz="0 0 0" rpy="0 0 0"/>
     <geometry>
-      <mesh filename="file://$(find robot)/meshes/wheel/base_link.stl" scale="0.001 0.001 0.001"/>
+      <mesh filename="file://$(find robot)/meshes/base_link.stl" scale="0.001 0.001 0.001"/>
     </geometry>
   </collision>
 </link>
-<joint name="chassis_joint" type="fixed">
-    <parent link="base_link"/>
-    <child link="chassis_link"/>
-    <origin xyz="-0.12 0 0.015"/>
-</joint>
+<link name="right_wheel">
+  <inertial>
+    <origin xyz="-1.7552218505301198e-06 0.027427365846597315 1.782423703911018e-07" rpy="0 0 0"/>
+    <mass value="0.05590599422944014"/>
+    <inertia ixx="3.2e-05" iyy="5e-05" izz="3.2e-05" ixy="-0.0" iyz="0.0" ixz="-0.0"/>
+  </inertial>
+  <visual>
+    <origin xyz="0.047514 -0.124767 0.077546" rpy="0 0 0"/>
+    <geometry>
+      <mesh filename="file://$(find robot)/meshes/Wheel_1_1.stl" scale="0.001 0.001 0.001"/>
+    </geometry>
+    <material name="silver"/>
+  </visual>
+  <collision>
+    <origin xyz="0.047514 -0.124767 0.077546" rpy="0 0 0"/>
+    <geometry>
+      <mesh filename="file://$(find robot)/meshes/Wheel_1_1.stl" scale="0.001 0.001 0.001"/>
+    </geometry>
+  </collision>
+</link>
+<link name="left_wheel">
+  <inertial>
+    <origin xyz="-1.7552218502803196e-06 -0.02742790766788944 1.5656025187382738e-07" rpy="0 0 0"/>
+    <mass value="0.05590599422944014"/>
+    <inertia ixx="3.2e-05" iyy="5e-05" izz="3.2e-05" ixy="0.0" iyz="0.0" ixz="0.0"/>
+  </inertial>
+  <visual>
+    <origin xyz="0.047514 0.122833 0.077546" rpy="0 0 0"/>
+    <geometry>
+      <mesh filename="file://$(find robot)/meshes/Wheel_2_1.stl" scale="0.001 0.001 0.001"/>
+    </geometry>
+    <material name="silver"/>
+  </visual>
+  <collision>
+    <origin xyz="0.047514 0.122833 0.077546" rpy="0 0 0"/>
+    <geometry>
+      <mesh filename="file://$(find robot)/meshes/Wheel_2_1.stl" scale="0.001 0.001 0.001"/>
+    </geometry>
+  </collision>
+</link>
 <joint name="right_wheel_joint" type="continuous">
-  <origin xyz="0.119 -0.1538 -0.059" rpy="0 0 0"/>
-  <parent link="chassis_link"/>
+  <origin xyz="-0.047514 0.124767 -0.077546" rpy="0 0 0"/>
+  <parent link="base_link"/>
   <child link="right_wheel"/>
-  <axis xyz="0 1 0"/>
+  <axis xyz="-0.0 1.0 0.0"/>
 </joint>
 <joint name="left_wheel_joint" type="continuous">
-  <origin xyz="0.119 -0.1538 0.059" rpy="0 0 0"/>
-  <parent link="chassis_link"/>
+  <origin xyz="-0.047514 -0.122833 -0.077546" rpy="0 0 0"/>
+  <parent link="base_link"/>
   <child link="left_wheel"/>
-  <axis xyz="0 -1 0"/>
+  <axis xyz="-0.0 -1.0 -0.0"/>
 </joint>
 </robot>

File: src/robot/urdf/robot_core.urdf.xacro (robot description, xacro)
@@ -2,6 +2,6 @@
 <robot name="rina" xmlns:xacro="http://www.ros.org/wiki/xacro" >
 <xacro:include filename="$(find robot)/urdf/robot.urdf.xacro" />
-<xacro:include filename="$(find robot)/urdf/sensors/lidar.xacro" />
-<!-- <xacro:include filename="$(find robot)/urdf/control/gazebo_control.xacro" /> -->
-<xacro:include filename="$(find robot)/urdf/control/ros2_control.xacro" />
+<!-- <xacro:include filename="$(find robot)/urdf/sensors/lidar.xacro" /> -->
+<xacro:include filename="$(find robot)/urdf/control/gazebo_control.xacro" />
+<!-- <xacro:include filename="$(find robot)/urdf/control/ros2_control.xacro" /> -->
 </robot>

File: src/robot/urdf/sensors/lidar.xacro (robot description, xacro)
@@ -10,5 +10,5 @@
   </inertial>
   <visual>
-    <origin xyz="0 0 0" rpy="0 0 0"/>
+    <origin xyz="0 0 0" rpy="0 0 ${pi}"/>
     <geometry>
       <mesh filename="file://$(find robot)/meshes/lidar/base_link.stl" scale="0.001 0.001 0.001"/>
@@ -17,5 +17,5 @@
   </visual>
   <collision>
-    <origin xyz="0 0 0" rpy="0 0 0"/>
+    <origin xyz="0 0 0" rpy="0 0 ${pi}"/>
     <geometry>
       <mesh filename="file://$(find robot)/meshes/lidar/base_link.stl" scale="0.001 0.001 0.001"/>
@@ -26,5 +26,5 @@
     <parent link="chassis_link"/>
     <child link="lidar_link"/>
-    <origin xyz="0 0 0" rpy="0 0 0"/>
+    <origin xyz="0.119 0 0.13" rpy="0 0 0"/>
 </joint>
 </robot>
