Commit message: added controllers, not working yet

File: src/robot/urdf/control/gazebo_control.xacro (robot description, xacro)
@@ -6,5 +6,5 @@
             <left_joint>left_wheel_joint</left_joint>
             <right_joint>right_wheel_joint</right_joint>
-            <wheel_separation>0.3048</wheel_separation>
+            <wheel_separation>0.325</wheel_separation>
             <wheel_diameter>0.07</wheel_diameter>
             <!-- Limits -->

File: src/robot/urdf/control/ros2_control.xacro (robot description, xacro)
@@ -1,35 +1,61 @@
 <?xml version="1.0"?>
 <robot xmlns:xacro="http://www.ros.org/wiki/xacro">
-    <ros2_control name="RealRobot" type="system">
-        <hardware>
-            <plugin>diffdrive_arduino/DiffDriveArduino</plugin>
-            <param name="left_wheel_name">left_wheel_joint</param>
-            <param name="right_wheel_name">right_wheel_joint</param>
-            <param name="loop_rate">30</param>
-            <param name="device">/dev/ttyACM0</param>
-            <param name="baud_rate">57600</param>
-            <param name="timeout">1000</param>
-            <param name="enc_counts_per_rev">560</param>
-        </hardware>
-        <joint name="left_wheel_joint">
-            <command_interface name="velocity">
-                <param name="min">-10</param>
-                <param name="max">10</param>
-            </command_interface>
-            <state_interface name="velocity"/>
-            <state_interface name="position"/>
-        </joint>
-        <joint name="right_wheel_joint">
-            <command_interface name="velocity">
-                <param name="min">-10</param>
-                <param name="max">10</param>
-            </command_interface>
-            <state_interface name="velocity"/>
-            <state_interface name="position"/>
-        </joint>
-    </ros2_control>
+    <xacro:unless value="$(arg sim_mode)">
+        <ros2_control name="RealRobot" type="system">
+            <hardware>
+                <plugin>diffdrive_arduino/DiffDriveArduino</plugin>
+                <param name="left_wheel_name">left_wheel_joint</param>
+                <param name="right_wheel_name">right_wheel_joint</param>
+                <param name="loop_rate">30</param>
+                <param name="device">/dev/ttyACM0</param>
+                <param name="baud_rate">57600</param>
+                <param name="timeout">1000</param>
+                <param name="enc_counts_per_rev">560</param>
+            </hardware>
+            <joint name="left_wheel_joint">
+                <command_interface name="velocity">
+                    <param name="min">-10</param>
+                    <param name="max">10</param>
+                </command_interface>
+                <state_interface name="velocity"/>
+                <state_interface name="position"/>
+            </joint>
+            <joint name="right_wheel_joint">
+                <command_interface name="velocity">
+                    <param name="min">-10</param>
+                    <param name="max">10</param>
+                </command_interface>
+                <state_interface name="velocity"/>
+                <state_interface name="position"/>
+            </joint>
+        </ros2_control>
+    </xacro:unless>
+    <xacro:if value="$(arg sim_mode)">
+        <ros2_control name="GazeboSystem" type="system">
+            <hardware>
+                <plugin>gazebo_ros2_control/GazeboSystem</plugin>
+            </hardware>
+            <joint name="left_wheel_joint">
+                <command_interface name="velocity">
+                    <param name="min">-10</param>
+                    <param name="max">10</param>
+                </command_interface>
+                <state_interface name="velocity"/>
+                <state_interface name="position"/>
+            </joint>
+            <joint name="right_wheel_joint">
+                <command_interface name="velocity">
+                    <param name="min">-10</param>
+                    <param name="max">10</param>
+                </command_interface>
+                <state_interface name="velocity"/>
+                <state_interface name="position"/>
+            </joint>
+        </ros2_control>
+    </xacro:if>
     <gazebo>
         <plugin name="gazebo_ros2_control" filename="libgazebo_ros2_control.so">
             <parameters>$(find robot)/config/controller.yaml</parameters>
+            <parameters>$(find robot)/config/gaz_control.yaml</parameters>
         </plugin>
     </gazebo>

File: src/robot/urdf/robot_core.urdf.xacro (robot description, xacro)
@@ -1,14 +1,13 @@
 <?xml version="1.0" ?>
 <robot name="rina" xmlns:xacro="http://www.ros.org/wiki/xacro" >
-<xacro:include filename="$(find robot)/urdf/robot.urdf.xacro" />
-<xacro:include filename="$(find robot)/urdf/sensors/lidar.xacro" />
-<xacro:include filename="$(find robot)/urdf/control/gazebo_control.xacro" />
-<!-- <xacro:include filename="$(find robot)/urdf/control/ros2_control.xacro" /> -->
-<!--
-<xacro:if value="$(arg use_ros2_control)">
-    <xacro:include filename="$(find robot)/urdf/control/ros2_control.xacro" />
-</xacro:if>
-<xacro:unless value="$(arg use_ros2_control)">
-    <xacro:include filename="$(find robot)/urdf/control/gazebo_control.xacro" />
-</xacro:unless> -->
+    <xacro:arg name="use_ros2_control" default="true"/>
+    <xacro:arg name="sim_mode" default="false"/>
+    <xacro:include filename="$(find robot)/urdf/robot.urdf.xacro" />
+    <xacro:include filename="$(find robot)/urdf/sensors/lidar.xacro" />
+    <xacro:if value="$(arg use_ros2_control)">
+        <xacro:include filename="$(find robot)/urdf/control/ros2_control.xacro" />
+    </xacro:if>
+    <xacro:unless value="$(arg use_ros2_control)">
+        <xacro:include filename="$(find robot)/urdf/control/gazebo_control.xacro" />
+    </xacro:unless>
 </robot>

File: src/robot/urdf/sensors/lidar.xacro (robot description, xacro)
@@ -8,5 +8,5 @@
     <parent link="base_link"/>
     <child link="lidar_link"/>
-    <origin xyz="0 0 0.13" rpy="0 0 0"/>
+    <origin xyz="-0.05 0 0.13" rpy="0 0 0"/>
 </joint>
 </robot>

Commit message: fixed odometry issues, however lots of things need improvement

File: src/robot/urdf/control/gazebo_control.xacro (robot description, xacro)
@@ -6,5 +6,5 @@
             <left_joint>left_wheel_joint</left_joint>
             <right_joint>right_wheel_joint</right_joint>
-            <wheel_separation>0.325</wheel_separation>
+            <wheel_separation>0.33</wheel_separation>
             <wheel_diameter>0.07</wheel_diameter>
             <!-- Limits -->

File: src/robot/urdf/materials.xacro (robot description, xacro)
@@ -1,4 +1,13 @@
 <?xml version="1.0" ?>
-<robot name="ros" xmlns:xacro="http://www.ros.org/wiki/xacro" >
+<robot xmlns:xacro="http://www.ros.org/wiki/xacro" >
+<material name="silver_default">
+  <color rgba="0.700 0.700 0.700 1.000"/>
+</material>
+<material name="rubber_soft">
+  <color rgba="0.15294117647058825 0.15294117647058825 0.15294117647058825 1.0"/>
+</material>
+<material name="plastic_glossy_grey">
+  <color rgba="0.7019607843137254 0.7019607843137254 0.7019607843137254 1.0"/>
+</material>
 <material name="silver">
   <color rgba="0.700 0.700 0.700 1.000"/>

File: src/robot/urdf/properties.xacro (robot description, xacro)
@@ -4,19 +4,19 @@
 <gazebo reference="base_link">
   <material>${body_color}</material>
+  <!-- <mu1>0.2</mu1>
+  <mu2>0.2</mu2>
+  <selfCollide>true</selfCollide>
+  <gravity>true</gravity> -->
+</gazebo>
+<gazebo reference="left_wheel_1">
+  <material>${body_color}</material>
   <mu1>0.2</mu1>
   <mu2>0.2</mu2>
-  <!-- <selfCollide>true</selfCollide>
-  <gravity>true</gravity> -->
-</gazebo>
-<gazebo reference="right_wheel">
-  <material>Gazebo/Black</material>
-  <!-- <mu1>0.2</mu1>
-  <mu2>0.2</mu2> -->
   <!-- <selfCollide>true</selfCollide> -->
 </gazebo>
-<gazebo reference="left_wheel">
-  <material>Gazebo/Black</material>
-  <!-- <mu1>0.2</mu1>
-  <mu2>0.2</mu2> -->
+<gazebo reference="right_wheel_1">
+  <material>${body_color}</material>
+  <mu1>0.2</mu1>
+  <mu2>0.2</mu2>
   <!-- <selfCollide>true</selfCollide> -->
 </gazebo>

File: src/robot/urdf/robot.urdf.xacro (robot description, xacro)
@@ -12,6 +12,6 @@
 <link name="base_link">
   <inertial>
-    <origin xyz="-0.07617652640143699 0.0009658129509204017 0.0007548948976041592" rpy="0 0 0"/>
-    <mass value="1.449043338359083"/>
+    <origin xyz="-0.028662948158421374 -9.161384338691405e-07 0.07830072749629308" rpy="0 0 0"/>
+    <mass value="1.4490433383590837"/>
     <inertia ixx="0.013382" iyy="0.012" izz="0.01271" ixy="-0.0" iyz="-0.0" ixz="-0.000167"/>
   </inertial>
@@ -21,5 +21,5 @@
       <mesh filename="file://$(find robot)/meshes/base_link.stl" scale="0.001 0.001 0.001"/>
     </geometry>
-    <material name="silver"/>
+    <material name="plastic_glossy_grey"/>
   </visual>
   <collision>
@@ -30,55 +30,129 @@
   </collision>
 </link>
-<link name="Wheel_1_1">
+<!-- <link name="left_wheel_1">
   <inertial>
-    <origin xyz="-1.7552218505301198e-06 0.027427365846597315 1.782423703911018e-07" rpy="0 0 0"/>
-    <mass value="0.05590599422944014"/>
+    <origin xyz="1.0883713637710694e-08 -0.027427636695222635 -2.1769573927273744e-06" rpy="0 0 0"/>
+    <mass value="0.05590599421880941"/>
     <inertia ixx="3.2e-05" iyy="5e-05" izz="3.2e-05" ixy="-0.0" iyz="0.0" ixz="-0.0"/>
   </inertial>
   <visual>
-    <origin xyz="0.047514 -0.124767 0.077546" rpy="0 0 0"/>
+    <origin xyz="-0.0 0.1238 0.0" rpy="0 0 0"/>
     <geometry>
-      <mesh filename="file://$(find robot)/meshes/Wheel_1_1.stl" scale="0.001 0.001 0.001"/>
+      <mesh filename="file://$(find robot)/meshes/left_wheel_1.stl" scale="0.001 0.001 0.001"/>
     </geometry>
-    <material name="silver"/>
+    <material name="rubber_soft"/>
   </visual>
   <collision>
-    <origin xyz="0.047514 -0.124767 0.077546" rpy="0 0 0"/>
+    <origin xyz="-0.0 0.1238 0.0" rpy="0 0 0"/>
     <geometry>
-      <mesh filename="file://$(find robot)/meshes/Wheel_1_1.stl" scale="0.001 0.001 0.001"/>
+      <mesh filename="file://$(find robot)/meshes/left_wheel_1.stl" scale="0.001 0.001 0.001"/>
     </geometry>
   </collision>
 </link>
-<link name="Wheel_2_1">
+<link name="right_wheel_1">
   <inertial>
-    <origin xyz="-1.7552218502803196e-06 -0.02742790766788944 1.5656025187382738e-07" rpy="0 0 0"/>
-    <mass value="0.05590599422944014"/>
-    <inertia ixx="3.2e-05" iyy="5e-05" izz="3.2e-05" ixy="0.0" iyz="0.0" ixz="0.0"/>
+    <origin xyz="-1.0841058577942398e-08 0.02742763675724355 -2.176978833869531e-06" rpy="0 0 0"/>
+    <mass value="0.055905994229440134"/>
+    <inertia ixx="3.2e-05" iyy="5e-05" izz="3.2e-05" ixy="-0.0" iyz="-0.0" ixz="0.0"/>
   </inertial>
   <visual>
-    <origin xyz="0.047514 0.122833 0.077546" rpy="0 0 0"/>
+    <origin xyz="0.0 -0.1238 -0.0" rpy="0 0 0"/>
     <geometry>
-      <mesh filename="file://$(find robot)/meshes/Wheel_2_1.stl" scale="0.001 0.001 0.001"/>
+      <mesh filename="file://$(find robot)/meshes/right_wheel_1.stl" scale="0.001 0.001 0.001"/>
     </geometry>
-    <material name="silver"/>
+    <material name="rubber_soft"/>
   </visual>
   <collision>
-    <origin xyz="0.047514 0.122833 0.077546" rpy="0 0 0"/>
+    <origin xyz="0.0 -0.1238 -0.0" rpy="0 0 0"/>
     <geometry>
-      <mesh filename="file://$(find robot)/meshes/Wheel_2_1.stl" scale="0.001 0.001 0.001"/>
+      <mesh filename="file://$(find robot)/meshes/right_wheel_1.stl" scale="0.001 0.001 0.001"/>
     </geometry>
   </collision>
-</link>
-<joint name="right_wheel_joint" type="continuous">
-  <origin xyz="-0.047514 0.124767 -0.077546" rpy="0 0 0"/>
+</link> -->
+<!-- <joint name="left_wheel_joint" type="continuous">
+  <origin xyz="0.0 -0.1238 0.0" rpy="0 0 0"/>
   <parent link="base_link"/>
-  <child link="Wheel_1_1"/>
+  <child link="left_wheel"/>
+  <origin xyz="0 ${wheel_offset_y} 0" rpy="-${pi/2} 0 0" />
   <axis xyz="0.0 1.0 0.0"/>
 </joint>
+<joint name="right_wheel_joint" type="continuous">
+  <origin xyz="0.0 0.1238 0.0" rpy="0 0 0"/>
+  <parent link="base_link"/>
+  <child link="right_wheel"/>
+  <axis xyz="0.0 1.0 0.0"/>
+  <origin xyz="0 ${-wheel_offset_y} 0" rpy="${pi/2} 0 0" />
+</joint> -->
+<xacro:property name="wheel_radius" value="0.035"/>
+<xacro:property name="wheel_thickness" value="0.04"/>
+<xacro:property name="wheel_mass" value="12.0"/>
+<xacro:property name="wheel_offset_x" value="0.226"/>
+<xacro:property name="wheel_offset_y" value="0.155"/>
+<xacro:property name="wheel_offset_z" value="0.01"/>
+<link name="left_wheel">
+    <visual>
+        <geometry>
+            <cylinder radius="${wheel_radius}" length="${wheel_thickness}"/>
+        </geometry>
+        <material name="blue"/>
+        <origin xyz="0 0 0" rpy="0 0 0"/>
+    </visual>
+    <collision>
+        <geometry>
+            <sphere radius="${wheel_radius}"/>
+        </geometry>
+    </collision>
+    <xacro:inertial_cylinder mass="${wheel_mass}" length="${wheel_thickness}" radius="${wheel_radius}">
+        <origin xyz="0 0 0" rpy="0 0 0"/>
+    </xacro:inertial_cylinder>
+</link>
+<link name="right_wheel">
+    <visual>
+        <geometry>
+            <cylinder radius="${wheel_radius}" length="${wheel_thickness}"/>
+        </geometry>
+        <material name="blue"/>
+    </visual>
+    <collision>
+        <geometry>
+            <sphere radius="${wheel_radius}"/>
+        </geometry>
+    </collision>
+    <xacro:inertial_cylinder mass="${wheel_mass}" length="${wheel_thickness}" radius="${wheel_radius}">
+        <origin xyz="0 0 0" rpy="0 0 0"/>
+    </xacro:inertial_cylinder>
+</link>
+<link name="counter_weight">
+    <visual>
+        <geometry>
+            <box size="0.03 0.04 0.05"/>
+        </geometry>
+        <material name="blue"/>
+    </visual>
+    <collision>
+        <geometry>
+            <box size="0.03 0.04 0.05"/>
+        </geometry>
+    </collision>
+    <xacro:inertial_box mass="1.0" x="0.03" y="0.04" z="0.05">
+      <origin xyz="${0.03/2} 0 ${0.05/2}" rpy="0 0 0"/>
+    </xacro:inertial_box>
+</link>
 <joint name="left_wheel_joint" type="continuous">
-  <origin xyz="-0.047514 -0.122833 -0.077546" rpy="0 0 0"/>
+    <parent link="base_link"/>
+    <child link="left_wheel"/>
+    <origin xyz="0 ${wheel_offset_y} 0" rpy="-${pi/2} 0 0" />
+    <axis xyz="0 0 1"/>
+</joint>
+<joint name="right_wheel_joint" type="continuous">
+    <parent link="base_link"/>
+    <child link="right_wheel"/>
+    <origin xyz="0 ${-wheel_offset_y} 0" rpy="${pi/2} 0 0" />
+    <axis xyz="0 0 -1"/>
+</joint>
+<joint name="counter_joint" type="fixed">
+  <origin xyz="-0.17 0.0 0.071" rpy="0.0 0.0 0.0"/>
   <parent link="base_link"/>
-  <child link="Wheel_2_1"/>
-  <axis xyz="0.0 1.0 0.0"/>
+  <child link="counter_weight"/>
 </joint>
 </robot>

File: src/robot/urdf/robot_core.urdf.xacro (robot description, xacro)
@@ -3,8 +3,8 @@
     <xacro:arg name="use_ros2_control" default="true"/>
     <xacro:arg name="sim_mode" default="false"/>
+    <xacro:include filename="$(find robot)/urdf/inertial_macros.xacro" />
     <xacro:include filename="$(find robot)/urdf/robot.urdf.xacro" />
-    <xacro:include filename="$(find robot)/urdf/inertial_macros.xacro" />
     <xacro:include filename="$(find robot)/urdf/sensors/lidar.xacro" />
-    <xacro:include filename="$(find robot)/urdf/sensors/camera.xacro" />
+    <!-- <xacro:include filename="$(find robot)/urdf/sensors/camera.xacro" /> -->
     <xacro:if value="$(arg use_ros2_control)">
         <xacro:include filename="$(find robot)/urdf/control/ros2_control.xacro" />

File: src/robot/urdf/sensors/lidar.xacro (robot description, xacro)
@@ -3,11 +3,28 @@
 <!-- <xacro:include filename="$(find robot)/urdf/materials.xacro" /> -->
 <!-- <xacro:include filename="$(find robot)/urdf/properties.xacro" /> -->
+<!--
 <link name="lidar_link">
-</link>
+</link> -->
 <joint name="laser_joint" type="fixed">
     <parent link="base_link"/>
-    <child link="lidar_link"/>
-    <origin xyz="-0.05 0 0.13" rpy="0 0 0"/>
+    <child link="laser_link"/>
+    <origin xyz="0.00 0 0.21" rpy="0 0 0"/>
 </joint>
+<link name="laser_link">
+    <visual>
+        <geometry>
+            <cylinder radius="0.05" length="0.04"/>
+        </geometry>
+        <material name="black"/>
+    </visual>
+    <collision>
+        <geometry>
+            <cylinder radius="0.05" length="0.04"/>
+        </geometry>
+    </collision>
+    <xacro:inertial_cylinder mass="0.05" length="0.03" radius="0.04">
+        <origin xyz="0 0 0" rpy="0 0 0"/>
+    </xacro:inertial_cylinder>
+</link>
 <gazebo reference="laser_link">
     <material>Gazebo/Black</material>
@@ -34,5 +51,5 @@
             </ros>
             <output_type>sensor_msgs/LaserScan</output_type>
-            <frame_name>lidar_link</frame_name>
+            <frame_name>laser_link</frame_name>
         </plugin>
     </sensor>
