Commit message: got lidar working with ydlidar_launch_view file

File: src/robot/urdf/properties.xacro (robot description, xacro)
@@ -21,5 +21,5 @@
   <!-- <selfCollide>true</selfCollide> -->
 </gazebo>
-<gazebo reference="lidar_link">
+<gazebo reference="laser_frame">
   <material>Gazebo/Black</material>
   <!-- <mu1>0.2</mu1> -->

File: src/robot/urdf/robot.urdf.xacro (robot description, xacro)
@@ -5,7 +5,7 @@
 <link name="base_link">
   <inertial>
-    <origin xyz="-0.0004442275486858486 -0.027763800307559608 0.04075489489760404" rpy="0 0 0"/>
+    <origin xyz="-0.07617652640143699 0.0009658129509204017 0.0007548948976041592" rpy="0 0 0"/>
     <mass value="1.449043338359083"/>
-    <inertia ixx="0.012" iyy="0.013382" izz="0.01271" ixy="0.0" iyz="-0.000167" ixz="0.0"/>
+    <inertia ixx="0.013382" iyy="0.012" izz="0.01271" ixy="-0.0" iyz="-0.0" ixz="-0.000167"/>
   </inertial>
   <visual>
@@ -23,55 +23,55 @@
   </collision>
 </link>
-<link name="right_wheel_1">
+<link name="Wheel_1_1">
   <inertial>
-    <origin xyz="-0.027427780444362282 -2.029127972526094e-06 1.7824236945435112e-07" rpy="0 0 0"/>
+    <origin xyz="-1.7552218505301198e-06 0.027427365846597315 1.782423703911018e-07" rpy="0 0 0"/>
     <mass value="0.05590599422944014"/>
-    <inertia ixx="5e-05" iyy="3.2e-05" izz="3.2e-05" ixy="0.0" iyz="-0.0" ixz="-0.0"/>
+    <inertia ixx="3.2e-05" iyy="5e-05" izz="3.2e-05" ixy="-0.0" iyz="0.0" ixz="-0.0"/>
   </inertial>
   <visual>
-    <origin xyz="0.124245 -0.000899 0.037546" rpy="0 0 0"/>
+    <origin xyz="0.047514 -0.124767 0.077546" rpy="0 0 0"/>
     <geometry>
-      <mesh filename="file://$(find robot)/meshes/right_wheel_1.stl" scale="0.001 0.001 0.001"/>
+      <mesh filename="file://$(find robot)/meshes/Wheel_1_1.stl" scale="0.001 0.001 0.001"/>
     </geometry>
     <material name="silver"/>
   </visual>
   <collision>
-    <origin xyz="0.124245 -0.000899 0.037546" rpy="0 0 0"/>
+    <origin xyz="0.047514 -0.124767 0.077546" rpy="0 0 0"/>
     <geometry>
-      <mesh filename="file://$(find robot)/meshes/right_wheel_1.stl" scale="0.001 0.001 0.001"/>
+      <mesh filename="file://$(find robot)/meshes/Wheel_1_1.stl" scale="0.001 0.001 0.001"/>
     </geometry>
   </collision>
 </link>
-<link name="left_wheel_1">
+<link name="Wheel_2_1">
   <inertial>
-    <origin xyz="0.027427493070124417 -2.0291279724919415e-06 1.5656025283833364e-07" rpy="0 0 0"/>
+    <origin xyz="-1.7552218502803196e-06 -0.02742790766788944 1.5656025187382738e-07" rpy="0 0 0"/>
     <mass value="0.05590599422944014"/>
-    <inertia ixx="5e-05" iyy="3.2e-05" izz="3.2e-05" ixy="-0.0" iyz="0.0" ixz="-0.0"/>
+    <inertia ixx="3.2e-05" iyy="5e-05" izz="3.2e-05" ixy="0.0" iyz="0.0" ixz="0.0"/>
   </inertial>
   <visual>
-    <origin xyz="-0.123355 -0.000899 0.037546" rpy="0 0 0"/>
+    <origin xyz="0.047514 0.122833 0.077546" rpy="0 0 0"/>
     <geometry>
-      <mesh filename="file://$(find robot)/meshes/left_wheel_1.stl" scale="0.001 0.001 0.001"/>
+      <mesh filename="file://$(find robot)/meshes/Wheel_2_1.stl" scale="0.001 0.001 0.001"/>
     </geometry>
     <material name="silver"/>
   </visual>
   <collision>
-    <origin xyz="-0.123355 -0.000899 0.037546" rpy="0 0 0"/>
+    <origin xyz="0.047514 0.122833 0.077546" rpy="0 0 0"/>
     <geometry>
-      <mesh filename="file://$(find robot)/meshes/left_wheel_1.stl" scale="0.001 0.001 0.001"/>
+      <mesh filename="file://$(find robot)/meshes/Wheel_2_1.stl" scale="0.001 0.001 0.001"/>
     </geometry>
   </collision>
 </link>
 <joint name="right_wheel_joint" type="continuous">
-  <origin xyz="-0.124245 0.000899 -0.037546" rpy="0 0 0"/>
+  <origin xyz="-0.047514 0.124767 -0.077546" rpy="0 0 0"/>
   <parent link="base_link"/>
-  <child link="right_wheel_1"/>
-  <axis xyz="-1.0 -0.0 -0.0"/>
+  <child link="Wheel_1_1"/>
+  <axis xyz="-0.0 1.0 0.0"/>
 </joint>
 <joint name="left_wheel_joint" type="continuous">
-  <origin xyz="0.123355 0.000899 -0.037546" rpy="0 0 0"/>
+  <origin xyz="-0.047514 -0.122833 -0.077546" rpy="0 0 0"/>
   <parent link="base_link"/>
-  <child link="left_wheel_1"/>
-  <axis xyz="1.0 -0.0 -0.0"/>
+  <child link="Wheel_2_1"/>
+  <axis xyz="-0.0 -1.0 -0.0"/>
 </joint>
 </robot>

File: src/robot/urdf/robot_core.urdf.xacro (robot description, xacro)
@@ -2,5 +2,5 @@
 <robot name="rina" xmlns:xacro="http://www.ros.org/wiki/xacro" >
 <xacro:include filename="$(find robot)/urdf/robot.urdf.xacro" />
-<!-- <xacro:include filename="$(find robot)/urdf/sensors/lidar.xacro" /> -->
+<xacro:include filename="$(find robot)/urdf/sensors/lidar.xacro" />
 <!-- <xacro:include filename="$(find robot)/urdf/control/gazebo_control.xacro" /> -->
 <xacro:include filename="$(find robot)/urdf/control/ros2_control.xacro" />

File: src/robot/urdf/sensors/lidar.xacro (robot description, xacro)
@@ -3,28 +3,10 @@
 <!-- <xacro:include filename="$(find robot)/urdf/materials.xacro" /> -->
 <!-- <xacro:include filename="$(find robot)/urdf/properties.xacro" /> -->
-<link name="lidar_link">
-  <inertial>
-    <origin xyz="-0.008294099570340205 -2.3249515286534618e-17 0.010701142222791043" rpy="0 0 0"/>
-    <mass value="0.18923752024949508"/>
-    <inertia ixx="8e-05" iyy="0.000141" izz="0.000162" ixy="0.0" iyz="-0.0" ixz="-2.4e-05"/>
-  </inertial>
-  <visual>
-    <origin xyz="0 0 0" rpy="0 0 ${pi}"/>
-    <geometry>
-      <mesh filename="file://$(find robot)/meshes/lidar/base_link.stl" scale="0.001 0.001 0.001"/>
-    </geometry>
-    <material name="silver"/>
-  </visual>
-  <collision>
-    <origin xyz="0 0 0" rpy="0 0 ${pi}"/>
-    <geometry>
-      <mesh filename="file://$(find robot)/meshes/lidar/base_link.stl" scale="0.001 0.001 0.001"/>
-    </geometry>
-  </collision>
+<link name="laser_frame">
 </link>
-<joint name="lidar_joint" type="fixed">
-    <parent link="chassis_link"/>
-    <child link="lidar_link"/>
-    <origin xyz="0.119 0 0.13" rpy="0 0 0"/>
+<joint name="laser_joint" type="fixed">
+    <parent link="base_link"/>
+    <child link="laser_frame"/>
+    <origin xyz="0 0 0.13" rpy="0 0 0"/>
 </joint>
 </robot>
