Commit message: slam toolbox parameters

File: src/robot/urdf/robot.urdf.xacro (robot description, xacro)
@@ -3,4 +3,11 @@
 <xacro:include filename="$(find robot)/urdf/materials.xacro" />
 <xacro:include filename="$(find robot)/urdf/properties.xacro" />
+<link name="base_footprint">
+</link>
+<joint name="footprint_joint" type="fixed">
+  <parent link="base_link"/>
+  <child link="base_footprint"/>
+  <origin xyz="0.0 0.0 0.0" rpy="0.0 0.0 0.0"/>
+</joint>
 <link name="base_link">
   <inertial>

File: src/robot/urdf/robot_core.urdf.xacro (robot description, xacro)
@@ -3,6 +3,6 @@
 <xacro:include filename="$(find robot)/urdf/robot.urdf.xacro" />
 <xacro:include filename="$(find robot)/urdf/sensors/lidar.xacro" />
-<!-- <xacro:include filename="$(find robot)/urdf/control/gazebo_control.xacro" /> -->
-<xacro:include filename="$(find robot)/urdf/control/ros2_control.xacro" />
+<xacro:include filename="$(find robot)/urdf/control/gazebo_control.xacro" />
+<!-- <xacro:include filename="$(find robot)/urdf/control/ros2_control.xacro" /> -->
 <!--
 <xacro:if value="$(arg use_ros2_control)">

File: src/robot/urdf/sensors/lidar.xacro (robot description, xacro)
@@ -3,9 +3,9 @@
 <!-- <xacro:include filename="$(find robot)/urdf/materials.xacro" /> -->
 <!-- <xacro:include filename="$(find robot)/urdf/properties.xacro" /> -->
-<link name="laser_frame">
+<link name="lidar_link">
 </link>
 <joint name="laser_joint" type="fixed">
     <parent link="base_link"/>
-    <child link="laser_frame"/>
+    <child link="lidar_link"/>
     <origin xyz="0 0 0.13" rpy="0 0 0"/>
 </joint>

Commit message: fixed wheel issue

File: src/robot/urdf/robot.urdf.xacro (robot description, xacro)
@@ -74,5 +74,5 @@
   <parent link="base_link"/>
   <child link="Wheel_1_1"/>
-  <axis xyz="-0.0 1.0 0.0"/>
+  <axis xyz="0.0 1.0 0.0"/>
 </joint>
 <joint name="left_wheel_joint" type="continuous">
@@ -80,5 +80,5 @@
   <parent link="base_link"/>
   <child link="Wheel_2_1"/>
-  <axis xyz="-0.0 -1.0 -0.0"/>
+  <axis xyz="0.0 1.0 0.0"/>
 </joint>
 </robot>

Commit message: made counter weight invisible by commenting out visual tag

File: src/robot/urdf/robot.urdf.xacro (robot description, xacro)
@@ -123,11 +123,12 @@
     </xacro:inertial_cylinder>
 </link>
+<!-- counter weight is invisible -->
 <link name="counter_weight">
-    <visual>
+    <!-- <visual>
         <geometry>
             <box size="0.03 0.04 0.05"/>
         </geometry>
         <material name="blue"/>
-    </visual>
+    </visual> -->
     <collision>
         <geometry>
