Commit message: fixed bad git structure

File: robot/urdf/control/gazebo_control.xacro (robot description, xacro)
@@ -6,5 +6,5 @@
             <left_joint>left_wheel_joint</left_joint>
             <right_joint>right_wheel_joint</right_joint>
-            <wheel_separation>0.33</wheel_separation>
+            <wheel_separation>0.32</wheel_separation>
             <wheel_diameter>0.07</wheel_diameter>
             <!-- Limits -->

File: robot/urdf/robot.urdf.xacro (robot description, xacro)
@@ -6,7 +6,7 @@
 </link>
 <joint name="footprint_joint" type="fixed">
+  <child link="base_footprint"/>
   <parent link="base_link"/>
-  <child link="base_footprint"/>
-  <origin xyz="0.0 0.0 0.0" rpy="0.0 0.0 0.0"/>
+  <origin xyz="0.0 0.0 -0.035" rpy="0.0 0.0 0.0"/>
 </joint>
 <link name="base_link">
@@ -86,8 +86,8 @@
 <xacro:property name="wheel_radius" value="0.035"/>
 <xacro:property name="wheel_thickness" value="0.04"/>
-<xacro:property name="wheel_mass" value="12.0"/>
-<xacro:property name="wheel_offset_x" value="0.226"/>
+<xacro:property name="wheel_mass" value="1.0"/>
+<!-- <xacro:property name="wheel_offset_x" value="0.226"/> -->
 <xacro:property name="wheel_offset_y" value="0.155"/>
-<xacro:property name="wheel_offset_z" value="0.01"/>
+<!-- <xacro:property name="wheel_offset_z" value="0.01"/> -->
 <link name="left_wheel">
     <visual>

File: robot/urdf/sensors/lidar.xacro (robot description, xacro)
@@ -8,8 +8,8 @@
 <joint name="laser_joint" type="fixed">
     <parent link="base_link"/>
-    <child link="laser_link"/>
+    <child link="laser_frame"/>
     <origin xyz="0.00 0 0.21" rpy="0 0 0"/>
 </joint>
-<link name="laser_link">
+<link name="laser_frame">
     <visual>
         <geometry>
@@ -27,5 +27,6 @@
     </xacro:inertial_cylinder>
 </link>
-<gazebo reference="laser_link">
+<!--
+<gazebo reference="laser_frame">
     <material>Gazebo/Black</material>
     <sensor name="laser" type="ray">
@@ -51,7 +52,7 @@
             </ros>
             <output_type>sensor_msgs/LaserScan</output_type>
-            <frame_name>laser_link</frame_name>
+            <frame_name>laser_frame</frame_name>
         </plugin>
     </sensor>
-</gazebo>
+</gazebo> -->
 </robot>
