Commit message: modified arduino comms, diff drive, urdf and controller yaml to include imu sensor but still in testing phase

File: robot/urdf/control/ros2_control.xacro (robot description, xacro)
@@ -29,4 +29,16 @@
                 <state_interface name="position"/>
             </joint>
+            <sensor name="imu_sensor">
+                <state_interface name="orientation.x"/>
+                <state_interface name="orientation.y"/>
+                <state_interface name="orientation.z"/>
+                <state_interface name="angular_velocity.x"/>
+                <state_interface name="angular_velocity.y"/>
+                <state_interface name="angular_velocity.z"/>
+                <state_interface name="linear_acceleration.x"/>
+                <state_interface name="linear_acceleration.y"/>
+                <state_interface name="linear_acceleration.z"/>
+                <param name="frame_id">imu_link</param>
+            </sensor>
         </ros2_control>
     </xacro:unless>

File: robot/urdf/robot.urdf.xacro (robot description, xacro)
@@ -140,4 +140,20 @@
     </xacro:inertial_box>
 </link>
+<link name="imu">
+    <!-- <visual>
+        <geometry>
+            <box size="0.03 0.04 0.05"/>
+        </geometry>
+        <material name="blue"/>
+    </visual> -->
+    <collision>
+        <geometry>
+            <box size="0.01 0.01 0.01"/>
+        </geometry>
+    </collision>
+    <xacro:inertial_box mass="1.0" x="0.01" y="0.01" z="0.01">
+      <origin xyz="${0.01/2} 0 ${0.01/2}" rpy="0 0 0"/>
+    </xacro:inertial_box>
+</link>
 <joint name="left_wheel_joint" type="continuous">
     <parent link="base_link"/>
@@ -157,3 +173,7 @@
   <child link="counter_weight"/>
 </joint>
+<joint name="imu_link" type="fixed">
+  <parent link="counter_weight"/>
+  <child link="imu"/>
+</joint>
 </robot>
