Commit message: modified urdf so you can now visualize imu data, also added convinient imu package to package list

File: robot/urdf/robot.urdf.xacro (robot description, xacro)
@@ -124,4 +124,21 @@
 </link>
 <!-- counter weight is invisible -->
+<link name="imu_link">
+    <!-- <visual>
+        <geometry>
+            <box size="0.03 0.04 0.05"/>
+        </geometry>
+        <material name="blue"/>
+    </visual> -->
+    <collision>
+        <geometry>
+            <box size="0.01 0.01 0.01"/>
+        </geometry>
+    </collision>
+    <xacro:inertial_box mass="1.0" x="0.01" y="0.01" z="0.01">
+      <origin xyz="${0.01/2} 0 ${0.01/2}" rpy="0 0 0"/>
+    </xacro:inertial_box>
+</link>
+<!-- counter weight is invisible -->
 <link name="counter_weight">
     <!-- <visual>
@@ -157,3 +174,8 @@
   <child link="counter_weight"/>
 </joint>
+<joint name="imu_joint" type="fixed">
+  <origin xyz="-0.17 0.0 0.071" rpy="0.0 0.0 0.0"/>
+  <parent link="counter_weight"/>
+  <child link="imu_link"/>
+</joint>
 </robot>

Commit message: added start of gazebo imu simulation, not yet tested

File: robot/urdf/robot.urdf.xacro (robot description, xacro)
@@ -124,21 +124,4 @@
 </link>
 <!-- counter weight is invisible -->
-<link name="imu_link">
-    <!-- <visual>
-        <geometry>
-            <box size="0.03 0.04 0.05"/>
-        </geometry>
-        <material name="blue"/>
-    </visual> -->
-    <collision>
-        <geometry>
-            <box size="0.01 0.01 0.01"/>
-        </geometry>
-    </collision>
-    <xacro:inertial_box mass="1.0" x="0.01" y="0.01" z="0.01">
-      <origin xyz="${0.01/2} 0 ${0.01/2}" rpy="0 0 0"/>
-    </xacro:inertial_box>
-</link>
-<!-- counter weight is invisible -->
 <link name="counter_weight">
     <!-- <visual>

File: robot/urdf/robot_core.urdf.xacro (robot description, xacro)
@@ -7,4 +7,5 @@
     <xacro:include filename="$(find robot)/urdf/sensors/lidar.xacro" />
     <xacro:include filename="$(find robot)/urdf/sensors/camera.xacro" />
+    <xacro:include filename="$(find robot)/urdf/sensors/imu.xacro" />
     <xacro:if value="$(arg use_ros2_control)">
         <xacro:include filename="$(find robot)/urdf/control/ros2_control.xacro" />

Commit message: fixed imu urdf bugs

File: robot/urdf/robot.urdf.xacro (robot description, xacro)
@@ -157,8 +157,3 @@
   <child link="counter_weight"/>
 </joint>
-<joint name="imu_joint" type="fixed">
-  <origin xyz="-0.17 0.0 0.071" rpy="0.0 0.0 0.0"/>
-  <parent link="counter_weight"/>
-  <child link="imu_link"/>
-</joint>
 </robot>

File: robot/urdf/robot_core.urdf.xacro (robot description, xacro)
@@ -7,5 +7,5 @@
     <xacro:include filename="$(find robot)/urdf/sensors/lidar.xacro" />
     <xacro:include filename="$(find robot)/urdf/sensors/camera.xacro" />
-    <xacro:include filename="$(find robot)/urdf/sensors/imu.xacro" />
+    <!-- <xacro:include filename="$(find robot)/urdf/sensors/imu.xacro" /> -->
     <xacro:if value="$(arg use_ros2_control)">
         <xacro:include filename="$(find robot)/urdf/control/ros2_control.xacro" />
