Commit message: fixed broken gazebo, added start of ekf, and added imu simulation, fixed camera as well

File: robot/urdf/properties.xacro (robot description, xacro)
@@ -1,5 +1,5 @@
 <?xml version="1.0" ?>
 <robot name="ros" xmlns:xacro="http://www.ros.org/wiki/xacro" >
-<xacro:property name="body_color" value="Gazebo/Silver" />
+<xacro:property name="body_color" value="Gazebo/Grey" />
 <gazebo reference="base_link">
   <material>${body_color}</material>

File: robot/urdf/sensors/camera.xacro (robot description, xacro)
@@ -4,5 +4,5 @@
         <parent link="base_link"/>
         <child link="camera_link"/>
-        <origin xyz="0.02 0 0.0" rpy="0 0 0"/>
+        <origin xyz="0.06 0 0.14" rpy="0 0 0"/>
     </joint>
     <link name="camera_link">

File: robot/urdf/sensors/imu.xacro (robot description, xacro)
@@ -22,16 +22,74 @@
     </xacro:inertial_box>
 </link>
-<!-- Will only run in Gazebo, make sure to put spherical data in Gazebo World file -->
-<sensor name="my_imu" type="imu">
-    <!-- ensure the sensor is active (required) -->
-    <always_on>true</always_on>
-    <update_rate>30</update_rate>
-    <plugin name="imu_plugin" filename="libgazebo_ros_imu_sensor.so">
-    <ros>
-        <!-- publish to /imu/data -->
-        <namespace>/imu</namespace>
-        <remapping>~/out:=data</remapping>
-    </ros>
-    </plugin>
-</sensor>
+<gazebo reference="imu_link">
+    <material>Gazebo/Black</material>
+    <!-- Will only run in Gazebo, make sure to put spherical data in Gazebo World file -->
+    <sensor name="imu_sensor" type="imu">
+        <!-- ensure the sensor is active (required) -->
+        <always_on>true</always_on>
+        <update_rate>30</update_rate>
+        <imu>
+          <angular_velocity>
+            <x>
+              <noise type="gaussian">
+                <mean>0.0</mean>
+                <stddev>2e-4</stddev>
+                <bias_mean>0.0000075</bias_mean>
+                <bias_stddev>0.0000008</bias_stddev>
+              </noise>
+            </x>
+            <y>
+              <noise type="gaussian">
+                <mean>0.0</mean>
+                <stddev>2e-4</stddev>
+                <bias_mean>0.0000075</bias_mean>
+                <bias_stddev>0.0000008</bias_stddev>
+              </noise>
+            </y>
+            <z>
+              <noise type="gaussian">
+                <mean>0.0</mean>
+                <stddev>2e-4</stddev>
+                <bias_mean>0.0000075</bias_mean>
+                <bias_stddev>0.0000008</bias_stddev>
+              </noise>
+            </z>
+          </angular_velocity>
+          <linear_acceleration>
+            <x>
+              <noise type="gaussian">
+                <mean>0.0</mean>
+                <stddev>1.7e-2</stddev>
+                <bias_mean>0.1</bias_mean>
+                <bias_stddev>0.001</bias_stddev>
+              </noise>
+            </x>
+            <y>
+              <noise type="gaussian">
+                <mean>0.0</mean>
+                <stddev>1.7e-2</stddev>
+                <bias_mean>0.1</bias_mean>
+                <bias_stddev>0.001</bias_stddev>
+              </noise>
+            </y>
+            <z>
+              <noise type="gaussian">
+                <mean>0.0</mean>
+                <stddev>1.7e-2</stddev>
+                <bias_mean>0.1</bias_mean>
+                <bias_stddev>0.001</bias_stddev>
+              </noise>
+            </z>
+          </linear_acceleration>
+        </imu>
+        <plugin name="imu_plugin" filename="libgazebo_ros_imu_sensor.so">
+            <ros>
+                <!-- publish to /imu/data -->
+                <namespace>/imu</namespace>
+                <remapping>~/out:=data</remapping>
+            </ros>
+            <frame_name>laser_frame</frame_name>
+        </plugin>
+    </sensor>
+</gazebo>
 </robot>
